Commit message: Created core URDF

File: description/robot.urdf.xacro (robot description, xacro)
@@ -2,3 +2,4 @@
 <robot xmlns:xacro="http://www.ros.org/wiki/xacro"  name="robot">
     <xacro:include filename="robot_core1.xacro" />
+    <xacro:include filename="gazebo_control.xacro" />
 </robot>

File: description/robot_core1.xacro (robot description, xacro)
@@ -40,4 +40,9 @@
         </xacro:inertial_box>
 	</link>
+    <gazebo reference="body_link">
+        <mu1>0.2</mu1>
+        <mu2>0.2</mu2>
+        <material>Gazebo/Red</material>
+    </gazebo>
 	<!-- End: Body link of the robot -->
 	<!-- START: Back right wheel of the robot and the joint -->
@@ -68,4 +73,9 @@
         </xacro:inertial_cylinder>
 	</link>
+    <gazebo reference="wheel1_link">
+        <mu1>0.2</mu1>
+        <mu2>0.2</mu2>
+        <material>Gazebo/Black</material>
+    </gazebo>
 	<!-- END: Back right wheel of the robot and the joint -->
 	<!-- START: Back left wheel of the robot and the joint -->
@@ -96,4 +106,9 @@
         </xacro:inertial_cylinder>
 	</link>
+    <gazebo reference="wheel2_link">
+        <mu1>0.2</mu1>
+        <mu2>0.2</mu2>
+        <material>Gazebo/Black</material>
+    </gazebo>
 	<!-- END: Back left wheel of the robot and the join -->
 	<!-- START: Front right wheel of the robot and the joint -->
@@ -124,4 +139,9 @@
         </xacro:inertial_cylinder>
 	</link>
+    <gazebo reference="wheel3_link">
+        <mu1>0.2</mu1>
+        <mu2>0.2</mu2>
+        <material>Gazebo/Black</material>
+    </gazebo>
 	<!-- END: Front right wheel of the robot and the joint -->
 	<!-- START: Front left wheel of the robot and joint -->
@@ -152,4 +172,9 @@
         </xacro:inertial_cylinder>
 	</link>
+    <gazebo reference="wheel4_link">
+        <mu1>0.2</mu1>
+        <mu2>0.2</mu2>
+        <material>Gazebo/Black</material>
+    </gazebo>
 	<!-- END: Front left wheel of the robot and joint -->
 </robot>
